File: _saved_arrowPad.sch (KiCad schematic (older format))
At the start: 24 parts, among them K1 KEYSW, K2 KEYSW, K3 KEYSW, K4 KEYSW, K5 KEYSW, K6 KEYSW, K7 KEYSW, K8 KEYSW, K9 KEYSW, SW1 SW_DIP_x01, U1 ProMicro, U2 NRF24L01_Breakout

Commit message: added drill holes
Parts:
- D10: footprint Connector_PinHeader_1.00mm:PinHeader_1x02_P1.00mm_Vertical -> Connector_PinHeader_2.54mm:PinHeader_1x02_P2.54mm_Vertical
Changed lines of the file:
@@
 F 0 "D10" V 7495 1529 50  0000 L CNN
 F 1 "LED" V 7586 1529 50  0000 L CNN
-F 2 "Connector_PinHeader_1.00mm:PinHeader_1x02_P1.00mm_Vertical" H 7550 1450 50  0001 C CNN
+F 2 "Connector_PinHeader_2.54mm:PinHeader_1x02_P2.54mm_Vertical" H 7550 1450 50  0001 C CNN
 F 3 "~" H 7550 1450 50  0001 C CNN
 	1    7550 1450
