File: arrowPad.sch (KiCad schematic (older format))
At the start: 22 parts, among them K1 KEYSW, K2 KEYSW, K3 KEYSW, K4 KEYSW, K5 KEYSW, K6 KEYSW, K7 KEYSW, K8 KEYSW, K9 KEYSW, SW1 SW_DIP_x01, U1 ProMicro, U2 NRF24L01_Breakout

Commit message: added ground plane
Parts:
- U1: footprint promicro:promicroreversetest2 -> promicro:proMicrov3
Changed lines of the file:
@@
 F 0 "U1" H 7800 4137 60  0000 C CNN
 F 1 "ProMicro" H 7800 4031 60  0000 C CNN
-F 2 "promicro:promicroreversetest2" H 7900 2050 60  0001 C CNN
+F 2 "promicro:proMicrov3" H 7900 2050 60  0001 C CNN
 F 3 "" H 7900 2050 60  0000 C CNN
 	1    7800 3100

Commit message: added wired communication between boards
Parts:
- added J1, J2: AudioJack3_Ground, symbol Connector:AudioJack3_Ground
- BT1: symbol Device:Battery_Cell -> arrowPad-rescue:Battery_Cell-Device
- D1, D2, D3, D4, D5, D6, D7, D8, D9: symbol Device:D -> arrowPad-rescue:D-Device
- K1, K2, K3, K4, K5, K6, K7, K8, K9: symbol keyboard_parts:KEYSW -> arrowPad-rescue:KEYSW-keyboard_parts
- SW1: symbol Switch:SW_DIP_x01 -> arrowPad-rescue:SW_DIP_x01-Switch
- U1: symbol promicro:ProMicro -> arrowPad-rescue:ProMicro-promicro
- U2: symbol RF:NRF24L01_Breakout -> arrowPad-rescue:NRF24L01_Breakout-RF
Connections:
- wire segments 38 -> 53
- no-connect marks 11 -> 9
Changed lines of the file:
@@
 $EndDescr
 $Comp
-L promicro:ProMicro U1
+L arrowPad-rescue:ProMicro-promicro U1
 U 1 1 5C46CD90
 P 7800 3100
@@
 $EndComp
 $Comp
-L keyboard_parts:KEYSW K3
+L arrowPad-rescue:KEYSW-keyboard_parts K3
 U 1 1 5C46CFB3
 P 5000 2400
@@
 $EndComp
 $Comp
-L Device:D D3
+L arrowPad-rescue:D-Device D3
 U 1 1 5C46D060
 P 4700 2550
@@
 $EndComp
 $Comp
-L Device:D D2
+L arrowPad-rescue:D-Device D2
 U 1 1 5C46FD83
 P 3950 2550
@@
 $EndComp
 $Comp
-L keyboard_parts:KEYSW K2
+L arrowPad-rescue:KEYSW-keyboard_parts K2
 U 1 1 5C46FDEC
 P 4250 2400
@@
 $EndComp
 $Comp
-L keyboard_parts:KEYSW K1
+L arrowPad-rescue:KEYSW-keyboard_parts K1
 U 1 1 5C46FEEC
 P 3500 2400
@@
 $EndComp
 $Comp
-L keyboard_parts:KEYSW K4
+L arrowPad-rescue:KEYSW-keyboard_parts K4
 U 1 1 5C47002C
 P 3500 3050
@@
 $EndComp
 $Comp
-L keyboard_parts:KEYSW K5
+L arrowPad-rescue:KEYSW-keyboard_parts K5
 U 1 1 5C4700D2
 P 4250 3050
@@
 $EndComp
 $Comp
-L keyboard_parts:KEYSW K6
+L arrowPad-rescue:KEYSW-keyboard_parts K6
 U 1 1 5C470147
 P 5000 3050
@@
 $EndComp
 $Comp
-L Device:D D1
+L arrowPad-rescue:D-Device D1
 U 1 1 5C470235
 P 3200 2550
@@
 $EndComp
 $Comp
-L Device:D D4
+L arrowPad-rescue:D-Device D4
 U 1 1 5C4703BA
 P 3200 3200
@@
 $EndComp
 $Comp
-L Device:D D5
+L arrowPad-rescue:D-Device D5
 U 1 1 5C470465
 P 3950 3200
@@
 $EndComp
 $Comp
-L Device:D D6
+L arrowPad-rescue:D-Device D6
 U 1 1 5C470513
 P 4700 3200
@@
 Col3
 $Comp
-L RF:NRF24L01_Breakout U2
+L arrowPad-rescue:NRF24L01_Breakout-RF U2
 U 1 1 5C47263D
 P 9550 3100
@@
 	9550 2500 9550 2350
 Wire Wire Line
-	9550 2350 8700 2350
+	9550 2350 8750 2350
 Wire Wire Line
 	8700 2350 8700 2650
@@
 GND1
 $Comp
-L Device:Battery_Cell BT1
+L arrowPad-rescue:Battery_Cell-Device BT1
 U 1 1 5C47463C
 P 9650 1650
@@
 $EndComp
 $Comp
-L keyboard_parts:KEYSW K7
+L arrowPad-rescue:KEYSW-keyboard_parts K7
 U 1 1 5C49C21E
 P 3500 3750
@@
 $EndComp
 $Comp
-L keyboard_parts:KEYSW K8
+L arrowPad-rescue:KEYSW-keyboard_parts K8
 U 1 1 5C49C30E
 P 4250 3750
@@
 $EndComp
 $Comp
-L keyboard_parts:KEYSW K9
+L arrowPad-rescue:KEYSW-keyboard_parts K9
 U 1 1 5C49C34C
 P 5000 3750
@@
 $EndComp
 $Comp
-L Device:D D7
+L arrowPad-rescue:D-Device D7
 U 1 1 5C49C727
 P 3200 3900
@@
 $EndComp
 $Comp
-L Device:D D8
+L arrowPad-rescue:D-Device D8
 U 1 1 5C49C7E5
 P 3950 3900
@@
 $EndComp
 $Comp
-L Device:D D9
+L arrowPad-rescue:D-Device D9
 U 1 1 5C49C9A6
 P 4700 3900
@@
 GND1
 NoConn ~ 9050 3400
-NoConn ~ 7100 2350
-NoConn ~ 7100 2450
 NoConn ~ 7100 2550
 NoConn ~ 7100 2650
@@
 NoConn ~ 7100 3450
 $Comp
-L Switch:SW_DIP_x01 SW1
+L arrowPad-rescue:SW_DIP_x01-Switch SW1
 U 1 1 5C52B630
 P 8900 1550
@@
 Wire Wire Line
 	9200 1450 9200 1550
+$Comp
+L Connector:AudioJack3_Ground J1
+U 1 1 5C63EF42
+P 6150 1700
+F 0 "J1" H 6130 2025 50  0000 C CNN
+F 1 "AudioJack3_Ground" H 6130 1934 50  0000 C CNN
+F 2 "" H 6150 1700 50  0001 C CNN
+F 3 "~" H 6150 1700 50  0001 C CNN
+	1    6150 1700
+	1    0    0    -1
+$EndComp
+$Comp
+L Connector:AudioJack3_Ground J2
+U 1 1 5C63F1CE
+P 5950 2750
+F 0 "J2" H 5930 3075 50  0000 C CNN
+F 1 "AudioJack3_Ground" H 5930 2984 50  0000 C CNN
+F 2 "" H 5950 2750 50  0001 C CNN
+F 3 "~" H 5950 2750 50  0001 C CNN
+	1    5950 2750
+	1    0    0    -1
+$EndComp
+Text Label 6150 2850 0    50   ~ 0
+RAW1
+Wire Wire Line
+	8750 2350 8750 1800
+Wire Wire Line
+	8750 1800 6350 1800
+Connection ~ 8750 2350
+Wire Wire Line
+	8750 2350 8700 2350
+Wire Wire Line
+	6350 1600 6950 1600
+Wire Wire Line
+	6950 1600 6950 2350
+Wire Wire Line
+	6950 2350 7100 2350
+Wire Wire Line
+	6950 2350 6650 2350
+Wire Wire Line
+	6650 2350 6650 2750
+Wire Wire Line
+	6650 2750 6150 2750
+Connection ~ 6950 2350
+Wire Wire Line
+	6350 1700 6800 1700
+Wire Wire Line
+	6800 1700 6800 2450
+Wire Wire Line
+	6800 2450 7100 2450
+Wire Wire Line
+	6800 2450 6350 2450
+Wire Wire Line
+	6350 2450 6350 2650
+Wire Wire Line
+	6350 2650 6150 2650
+Connection ~ 6800 2450
 $EndSCHEMATC

Commit message: final v1
Parts:
- removed SW1: SW_DIP_x01, Connector_PinHeader_2.54mm:PinHeader_1x02_P2.54mm_Vertical, symbol arrowPad-rescue:SW_DIP_x01-Switch
- added D10: LED, Connector_PinHeader_2.54mm:PinHeader_1x02_P2.54mm_Vertical, symbol Device:LED
- added R1: R, keyboard_parts:D_SOD123_axial, symbol Device:R
- added U3: ADG417BN, Connector_PinHeader_2.54mm:PinHeader_1x03_P2.54mm_Vertical, symbol Analog_Switch:ADG417BN
- J1, J2: footprint (none) -> Connector_PinHeader_2.54mm:PinHeader_1x04_P2.54mm_Vertical; symbol Connector:AudioJack3_Ground -> arrowPad-rescue:AudioJack3_Ground-Connector
- U1: footprint promicro:proMicrov3 -> Transformer_SMD:proMicrov6
Connections:
- wire segments 53 -> 58
- no-connect marks 9 -> 8
Changed lines of the file:
@@
 F 0 "U1" H 7800 4137 60  0000 C CNN
 F 1 "ProMicro" H 7800 4031 60  0000 C CNN
-F 2 "promicro:proMicrov3" H 7900 2050 60  0001 C CNN
+F 2 "Transformer_SMD:proMicrov6" H 7900 2050 60  0001 C CNN
 F 3 "" H 7900 2050 60  0000 C CNN
 	1    7800 3100
@@
 Wire Wire Line
 	8550 2950 8550 3300
-Text Label 7100 2950 2    50   ~ 0
+Text Label 7100 2850 2    50   ~ 0
 Col1
 Text Label 7100 3050 2    50   ~ 0
@@
 Text Label 8500 2350 0    50   ~ 0
 RAW1
-Text Label 8600 1550 2    50   ~ 0
+Text Label 8200 1450 3    50   ~ 0
 RAW1
 Text Label 9650 1750 0    50   ~ 0
@@
 NoConn ~ 7100 2650
 NoConn ~ 7100 2750
-NoConn ~ 7100 2850
 NoConn ~ 8500 2850
 NoConn ~ 8500 2750
 NoConn ~ 8500 2550
 NoConn ~ 7100 3450
-$Comp
-L arrowPad-rescue:SW_DIP_x01-Switch SW1
-U 1 1 5C52B630
-P 8900 1550
-F 0 "SW1" H 8900 1817 50  0000 C CNN
-F 1 "SW_DIP_x01" H 8900 1726 50  0000 C CNN
-F 2 "Connector_PinHeader_2.54mm:PinHeader_1x02_P2.54mm_Vertical" H 8900 1550 50  0001 C CNN
-F 3 "" H 8900 1550 50  0001 C CNN
-	1    8900 1550
-	1    0    0    -1
-$EndComp
 Wire Wire Line
 	9650 1450 9200 1450
@@
 	9200 1450 9200 1550
 $Comp
-L Connector:AudioJack3_Ground J1
+L arrowPad-rescue:AudioJack3_Ground-Connector J1
 U 1 1 5C63EF42
 P 6150 1700
 F 0 "J1" H 6130 2025 50  0000 C CNN
 F 1 "AudioJack3_Ground" H 6130 1934 50  0000 C CNN
-F 2 "" H 6150 1700 50  0001 C CNN
+F 2 "Connector_PinHeader_2.54mm:PinHeader_1x04_P2.54mm_Vertical" H 6150 1700 50  0001 C CNN
 F 3 "~" H 6150 1700 50  0001 C CNN
 	1    6150 1700
@@
 $EndComp
 $Comp
-L Connector:AudioJack3_Ground J2
+L arrowPad-rescue:AudioJack3_Ground-Connector J2
 U 1 1 5C63F1CE
 P 5950 2750
 F 0 "J2" H 5930 3075 50  0000 C CNN
 F 1 "AudioJack3_Ground" H 5930 2984 50  0000 C CNN
-F 2 "" H 5950 2750 50  0001 C CNN
+F 2 "Connector_PinHeader_2.54mm:PinHeader_1x04_P2.54mm_Vertical" H 5950 2750 50  0001 C CNN
 F 3 "~" H 5950 2750 50  0001 C CNN
 	1    5950 2750
@@
 	6350 2650 6150 2650
 Connection ~ 6800 2450
+$Comp
+L Device:R R1
+U 1 1 5C64D075
+P 6450 3500
+F 0 "R1" H 6520 3546 50  0000 L CNN
+F 1 "R" H 6520 3455 50  0000 L CNN
+F 2 "keyboard_parts:D_SOD123_axial" V 6380 3500 50  0001 C CNN
+F 3 "~" H 6450 3500 50  0001 C CNN
+	1    6450 3500
+	1    0    0    -1
+$EndComp
+$Comp
+L Device:LED D10
+U 1 1 5C64D1AE
+P 6450 4000
+F 0 "D10" V 6488 3882 50  0000 R CNN
+F 1 "LED" V 6397 3882 50  0000 R CNN
+F 2 "Connector_PinHeader_2.54mm:PinHeader_1x02_P2.54mm_Vertical" H 6450 4000 50  0001 C CNN
+F 3 "~" H 6450 4000 50  0001 C CNN
+	1    6450 4000
+	0    -1   -1   0
+$EndComp
+Text Label 6450 4150 2    50   ~ 0
+GND1
+Wire Wire Line
+	6450 3850 6450 3650
+Wire Wire Line
+	6450 3350 6450 2950
+Wire Wire Line
+	6450 2950 7100 2950
+Wire Wire Line
+	9200 1550 8500 1550
+Wire Wire Line
+	8500 1550 8500 1250
+$Comp
+L Analog_Switch:ADG417BN U3
+U 1 1 5C659A57
+P 8200 1250
+F 0 "U3" H 8200 1517 50  0000 C CNN
+F 1 "ADG417BN" H 8200 1426 50  0000 C CNN
+F 2 "Connector_PinHeader_2.54mm:PinHeader_1x03_P2.54mm_Vertical" H 8200 1150 50  0001 C CNN
+F 3 "http://www.analog.com/media/en/technical-documentation/data-sheets/ADG417.pdf" H 8200 1250 50  0001 C CNN
+	1    8200 1250
+	1    0    0    -1
+$EndComp
 $EndSCHEMATC
