File: pcb_files/_saved_arrowPad.sch (KiCad schematic (older format))
At the start: 60 parts, among them J1 AudioJack3_Ground, J2 AudioJack3_Ground, K1 KEYSW, K10 KEYSW, K11 KEYSW, K12 KEYSW, K13 KEYSW, K14 KEYSW, K15 KEYSW, K16 KEYSW, K2 KEYSW, K3 KEYSW, K4 KEYSW, K5 KEYSW, K6 KEYSW, K7 KEYSW, K8 KEYSW, K9 KEYSW, U1 ProMicro, U2 NRF24L01_Breakout, U3 ADG417BN, U4 AMS1117-3.3, U5 ADG417BN, U6 ADG417BN, U7 TLC5940PWP

Commit message: TLC5940 LED controller
Parts:
- BT1: footprint keyboard_parts:C_3528 -> Connector_PinHeader_2.54mm:PinHeader_1x02_P2.54mm_Vertical
- D21: value 21 -> LED
- J1, J2: footprint foots:CUI_SJ1-3514-SMT[PAD1,2,34]Backside -> foots:CUI_SJ-43514-SMT(1,2,3,4reverseside)
Changed lines of the file:
@@
 F 0 "BT1" H 9768 1746 50  0000 L CNN
 F 1 "Battery_Cell" H 9768 1655 50  0000 L CNN
-F 2 "keyboard_parts:C_3528" V 9650 1710 50  0001 C CNN
+F 2 "Connector_PinHeader_2.54mm:PinHeader_1x02_P2.54mm_Vertical" V 9650 1710 50  0001 C CNN
 F 3 "~" V 9650 1710 50  0001 C CNN
 	1    9650 1650
@@
 F 0 "J1" H 5580 2375 50  0000 C CNN
 F 1 "AudioJack3_Ground" H 5580 2284 50  0000 C CNN
-F 2 "foots:CUI_SJ1-3514-SMT[PAD1,2,34]Backside" H 5600 2050 50  0001 C CNN
+F 2 "foots:CUI_SJ-43514-SMT(1,2,3,4reverseside)" H 5600 2050 50  0001 C CNN
 F 3 "~" H 5600 2050 50  0001 C CNN
 	1    5600 2050
@@
 F 0 "J2" H 5530 3175 50  0000 C CNN
 F 1 "AudioJack3_Ground" H 5530 3084 50  0000 C CNN
-F 2 "foots:CUI_SJ1-3514-SMT[PAD1,2,34]Backside" H 5550 2850 50  0001 C CNN
+F 2 "foots:CUI_SJ-43514-SMT(1,2,3,4reverseside)" H 5550 2850 50  0001 C CNN
 F 3 "~" H 5550 2850 50  0001 C CNN
 	1    5550 2850
@@
 P 6600 5000
 F 0 "D21" V 6545 5079 50  0000 L CNN
-F 1 "21" V 6636 5079 50  0000 L CNN
+F 1 "LED" V 6636 5079 50  0000 L CNN
 F 2 "keyboard_parts:C_3528" H 6600 5000 50  0001 C CNN
 F 3 "~" H 6600 5000 50  0001 C CNN

Commit message: traces from led ic
Parts:
- D1: footprint keyboard_parts:C_3528 -> keyboard_parts:D_SOD123_axial
- D20, D21, D22, D23, D24, D25, D26, D27, D28, D29, D30, D31, D32, D33, D34, D35: footprint keyboard_parts:C_3528 -> foots:C_3528v1
- J1, J2: footprint foots:CUI_SJ-43514-SMT(1,2,3,4reverseside) -> SJ-43514-SMT:CUI_SJ-43514-SMT
Changed lines of the file:
@@
 F 0 "D1" V 1746 1921 50  0000 R CNN
 F 1 "D" V 1655 1921 50  0000 R CNN
-F 2 "keyboard_parts:C_3528" H 1700 2000 50  0001 C CNN
+F 2 "keyboard_parts:D_SOD123_axial" H 1700 2000 50  0001 C CNN
 F 3 "~" H 1700 2000 50  0001 C CNN
 	1    1700 2000
@@
 F 0 "J1" H 5580 2375 50  0000 C CNN
 F 1 "AudioJack3_Ground" H 5580 2284 50  0000 C CNN
-F 2 "foots:CUI_SJ-43514-SMT(1,2,3,4reverseside)" H 5600 2050 50  0001 C CNN
+F 2 "SJ-43514-SMT:CUI_SJ-43514-SMT" H 5600 2050 50  0001 C CNN
 F 3 "~" H 5600 2050 50  0001 C CNN
 	1    5600 2050
@@
 F 0 "J2" H 5530 3175 50  0000 C CNN
 F 1 "AudioJack3_Ground" H 5530 3084 50  0000 C CNN
-F 2 "foots:CUI_SJ-43514-SMT(1,2,3,4reverseside)" H 5550 2850 50  0001 C CNN
+F 2 "SJ-43514-SMT:CUI_SJ-43514-SMT" H 5550 2850 50  0001 C CNN
 F 3 "~" H 5550 2850 50  0001 C CNN
 	1    5550 2850
@@
 F 0 "D20" V 6845 5079 50  0000 L CNN
 F 1 "LED" V 6936 5079 50  0000 L CNN
-F 2 "keyboard_parts:C_3528" H 6900 5000 50  0001 C CNN
+F 2 "foots:C_3528v1" H 6900 5000 50  0001 C CNN
 F 3 "~" H 6900 5000 50  0001 C CNN
 	1    6900 5000
@@
 F 0 "D21" V 6545 5079 50  0000 L CNN
 F 1 "LED" V 6636 5079 50  0000 L CNN
-F 2 "keyboard_parts:C_3528" H 6600 5000 50  0001 C CNN
+F 2 "foots:C_3528v1" H 6600 5000 50  0001 C CNN
 F 3 "~" H 6600 5000 50  0001 C CNN
 	1    6600 5000
@@
 F 0 "D22" V 6245 5079 50  0000 L CNN
 F 1 "LED" V 6336 5079 50  0000 L CNN
-F 2 "keyboard_parts:C_3528" H 6300 5000 50  0001 C CNN
+F 2 "foots:C_3528v1" H 6300 5000 50  0001 C CNN
 F 3 "~" H 6300 5000 50  0001 C CNN
 	1    6300 5000
@@
 F 0 "D23" V 5945 5079 50  0000 L CNN
 F 1 "LED" V 6036 5079 50  0000 L CNN
-F 2 "keyboard_parts:C_3528" H 6000 5000 50  0001 C CNN
+F 2 "foots:C_3528v1" H 6000 5000 50  0001 C CNN
 F 3 "~" H 6000 5000 50  0001 C CNN
 	1    6000 5000
@@
 F 0 "D24" V 5645 5079 50  0000 L CNN
 F 1 "LED" V 5736 5079 50  0000 L CNN
-F 2 "keyboard_parts:C_3528" H 5700 5000 50  0001 C CNN
+F 2 "foots:C_3528v1" H 5700 5000 50  0001 C CNN
 F 3 "~" H 5700 5000 50  0001 C CNN
 	1    5700 5000
@@
 F 0 "D25" V 5345 5079 50  0000 L CNN
 F 1 "LED" V 5436 5079 50  0000 L CNN
-F 2 "keyboard_parts:C_3528" H 5400 5000 50  0001 C CNN
+F 2 "foots:C_3528v1" H 5400 5000 50  0001 C CNN
 F 3 "~" H 5400 5000 50  0001 C CNN
 	1    5400 5000
@@
 F 0 "D26" V 5045 5079 50  0000 L CNN
 F 1 "LED" V 5136 5079 50  0000 L CNN
-F 2 "keyboard_parts:C_3528" H 5100 5000 50  0001 C CNN
+F 2 "foots:C_3528v1" H 5100 5000 50  0001 C CNN
 F 3 "~" H 5100 5000 50  0001 C CNN
 	1    5100 5000
@@
 F 0 "D27" V 4745 5079 50  0000 L CNN
 F 1 "LED" V 4836 5079 50  0000 L CNN
-F 2 "keyboard_parts:C_3528" H 4800 5000 50  0001 C CNN
+F 2 "foots:C_3528v1" H 4800 5000 50  0001 C CNN
 F 3 "~" H 4800 5000 50  0001 C CNN
 	1    4800 5000
@@
 F 0 "D28" V 4445 5079 50  0000 L CNN
 F 1 "LED" V 4536 5079 50  0000 L CNN
-F 2 "keyboard_parts:C_3528" H 4500 5000 50  0001 C CNN
+F 2 "foots:C_3528v1" H 4500 5000 50  0001 C CNN
 F 3 "~" H 4500 5000 50  0001 C CNN
 	1    4500 5000
@@
 F 0 "D29" V 4145 5079 50  0000 L CNN
 F 1 "LED" V 4236 5079 50  0000 L CNN
-F 2 "keyboard_parts:C_3528" H 4200 5000 50  0001 C CNN
+F 2 "foots:C_3528v1" H 4200 5000 50  0001 C CNN
 F 3 "~" H 4200 5000 50  0001 C CNN
 	1    4200 5000
@@
 F 0 "D30" V 3845 5079 50  0000 L CNN
 F 1 "LED" V 3936 5079 50  0000 L CNN
-F 2 "keyboard_parts:C_3528" H 3900 5000 50  0001 C CNN
+F 2 "foots:C_3528v1" H 3900 5000 50  0001 C CNN
 F 3 "~" H 3900 5000 50  0001 C CNN
 	1    3900 5000
@@
 F 0 "D31" V 3545 5079 50  0000 L CNN
 F 1 "LED" V 3636 5079 50  0000 L CNN
-F 2 "keyboard_parts:C_3528" H 3600 5000 50  0001 C CNN
+F 2 "foots:C_3528v1" H 3600 5000 50  0001 C CNN
 F 3 "~" H 3600 5000 50  0001 C CNN
 	1    3600 5000
@@
 F 0 "D32" V 3245 5079 50  0000 L CNN
 F 1 "LED" V 3336 5079 50  0000 L CNN
-F 2 "keyboard_parts:C_3528" H 3300 5000 50  0001 C CNN
+F 2 "foots:C_3528v1" H 3300 5000 50  0001 C CNN
 F 3 "~" H 3300 5000 50  0001 C CNN
 	1    3300 5000
@@
 F 0 "D33" V 2945 5079 50  0000 L CNN
 F 1 "LED" V 3036 5079 50  0000 L CNN
-F 2 "keyboard_parts:C_3528" H 3000 5000 50  0001 C CNN
+F 2 "foots:C_3528v1" H 3000 5000 50  0001 C CNN
 F 3 "~" H 3000 5000 50  0001 C CNN
 	1    3000 5000
@@
 F 0 "D34" V 2645 5079 50  0000 L CNN
 F 1 "LED" V 2736 5079 50  0000 L CNN
-F 2 "keyboard_parts:C_3528" H 2700 5000 50  0001 C CNN
+F 2 "foots:C_3528v1" H 2700 5000 50  0001 C CNN
 F 3 "~" H 2700 5000 50  0001 C CNN
 	1    2700 5000
@@
 F 0 "D35" V 2345 5079 50  0000 L CNN
 F 1 "LED" V 2436 5079 50  0000 L CNN
-F 2 "keyboard_parts:C_3528" H 2400 5000 50  0001 C CNN
+F 2 "foots:C_3528v1" H 2400 5000 50  0001 C CNN
 F 3 "~" H 2400 5000 50  0001 C CNN
 	1    2400 5000
