File: pcb_files/arrowPad.sch (KiCad schematic (older format))
At the start: 26 parts, among them J1 AudioJack3_Ground, J2 AudioJack3_Ground, K1 KEYSW, K2 KEYSW, K3 KEYSW, K4 KEYSW, K5 KEYSW, K6 KEYSW, K7 KEYSW, K8 KEYSW, K9 KEYSW, U1 ProMicro, U2 NRF24L01_Breakout, U3 ADG417BN

Commit message: updated schem
Parts:
- added U4: AMS1117-3.3, promicro:AMS1117flipped, symbol AMS1117-3.3:AMS1117-3.3
- J1, J2: footprint Connector_PinHeader_2.54mm:PinHeader_1x04_P2.54mm_Vertical -> SJ1-3514-SMT:CUI_SJ1-3514-SMT
Connections:
- wire segments 58 -> 62
Changed lines of the file:
@@
 Row3
-Wire Wire Line
-	9550 2500 9550 2350
 Wire Wire Line
 	9550 2350 8750 2350
@@
 F 0 "J1" H 6130 2025 50  0000 C CNN
 F 1 "AudioJack3_Ground" H 6130 1934 50  0000 C CNN
-F 2 "Connector_PinHeader_2.54mm:PinHeader_1x04_P2.54mm_Vertical" H 6150 1700 50  0001 C CNN
+F 2 "SJ1-3514-SMT:CUI_SJ1-3514-SMT" H 6150 1700 50  0001 C CNN
 F 3 "~" H 6150 1700 50  0001 C CNN
 	1    6150 1700
@@
 F 0 "J2" H 5930 3075 50  0000 C CNN
 F 1 "AudioJack3_Ground" H 5930 2984 50  0000 C CNN
-F 2 "Connector_PinHeader_2.54mm:PinHeader_1x04_P2.54mm_Vertical" H 5950 2750 50  0001 C CNN
+F 2 "SJ1-3514-SMT:CUI_SJ1-3514-SMT" H 5950 2750 50  0001 C CNN
 F 3 "~" H 5950 2750 50  0001 C CNN
 	1    5950 2750
@@
 	1    0    0    -1
 $EndComp
+$Comp
+L AMS1117-3.3:AMS1117-3.3 U4
+U 1 1 5C962AD9
+P 10200 2200
+F 0 "U4" H 10200 2567 50  0000 C CNN
+F 1 "AMS1117-3.3" H 10200 2476 50  0000 C CNN
+F 2 "promicro:AMS1117flipped" H 10200 2200 50  0001 L BNN
+F 3 "Sot223/Pkg 1-Amp 3.3-Volt Low Drop Out Voltage Regulatator" H 10200 2200 50  0001 L BNN
+F 4 "Advanced Monolithic Systems" H 10200 2200 50  0001 L BNN "Field4"
+F 5 "None" H 10200 2200 50  0001 L BNN "Field5"
+F 6 "Unavailable" H 10200 2200 50  0001 L BNN "Field6"
+F 7 "None" H 10200 2200 50  0001 L BNN "Field7"
+F 8 "AMS1117-3.3" H 10200 2200 50  0001 L BNN "Field8"
+	1    10200 2200
+	1    0    0    -1
+$EndComp
+Wire Wire Line
+	9550 2350 9550 2100
+Wire Wire Line
+	9550 2100 9600 2100
+Wire Wire Line
+	10800 2100 11000 2100
+Wire Wire Line
+	11000 2100 11000 2500
+Wire Wire Line
+	11000 2500 9550 2500
+Text Label 10800 2300 0    50   ~ 0
+GND1
 $EndSCHEMATC

Commit message: v2
Parts:
- removed D10: LED, Connector_PinHeader_2.54mm:PinHeader_1x02_P2.54mm_Vertical, symbol Device:LED
- removed R1: R, keyboard_parts:D_SOD123_axial, symbol Device:R
- added D12, D13, D14, D15, D16, D4, D8: D, keyboard_parts:D_SOD123_axial, symbol arrowPad-rescue:D-Device
- added K12, K13, K14, K15, K16, K4, K8: KEYSW, keyswitches:PG1350_socket, symbol arrowPad-rescue:KEYSW-keyboard_parts
- J1, J2: footprint SJ1-3514-SMT:CUI_SJ1-3514-SMT -> foots:CUI_SJ1-3514-SMT[PAD1,2,34]
- U1: footprint Transformer_SMD:proMicrov6 -> promicro:ProMicro
- renumbered D8 to D10, D9 to D11, D4 to D5, D5 to D6, D6 to D7, D7 to D9, K8 to K10, K9 to K11, K4 to K5, K5 to K6, K6 to K7, K7 to K9
Connections:
- net labels added: Col4, Row4, VCC1
- wire segments 62 -> 65
- no-connect marks 8 -> 10

Commit message: updated
Parts:
- added R? (x2): R, symbol Device:R
- added U?: ADG417BN, Connector_PinHeader_2.54mm:PinHeader_1x03_P2.54mm_Vertical, symbol Analog_Switch:ADG417BN
Connections:
- wire segments 65 -> 68
Changed lines of the file:
@@
 L arrowPad-rescue:AudioJack3_Ground-Connector J1
 U 1 1 5C63EF42
-P 5950 2000
-F 0 "J1" H 5930 2325 50  0000 C CNN
-F 1 "AudioJack3_Ground" H 5930 2234 50  0000 C CNN
-F 2 "foots:CUI_SJ1-3514-SMT[PAD1,2,34]" H 5950 2000 50  0001 C CNN
-F 3 "~" H 5950 2000 50  0001 C CNN
-	1    5950 2000
+P 5600 2050
+F 0 "J1" H 5580 2375 50  0000 C CNN
+F 1 "AudioJack3_Ground" H 5580 2284 50  0000 C CNN
+F 2 "foots:CUI_SJ1-3514-SMT[PAD1,2,34]" H 5600 2050 50  0001 C CNN
+F 3 "~" H 5600 2050 50  0001 C CNN
+	1    5600 2050
 	1    0    0    -1
 $EndComp
@@
 L arrowPad-rescue:AudioJack3_Ground-Connector J2
 U 1 1 5C63F1CE
-P 5950 2750
-F 0 "J2" H 5930 3075 50  0000 C CNN
-F 1 "AudioJack3_Ground" H 5930 2984 50  0000 C CNN
-F 2 "foots:CUI_SJ1-3514-SMT[PAD1,2,34]" H 5950 2750 50  0001 C CNN
-F 3 "~" H 5950 2750 50  0001 C CNN
-	1    5950 2750
-	1    0    0    -1
-$EndComp
-Text Label 6150 2850 0    50   ~ 0
+P 5550 2850
+F 0 "J2" H 5530 3175 50  0000 C CNN
+F 1 "AudioJack3_Ground" H 5530 3084 50  0000 C CNN
+F 2 "foots:CUI_SJ1-3514-SMT[PAD1,2,34]" H 5550 2850 50  0001 C CNN
+F 3 "~" H 5550 2850 50  0001 C CNN
+	1    5550 2850
+	1    0    0    -1
+$EndComp
+Text Label 5750 2950 0    50   ~ 0
 RAW1
 Wire Wire Line
@@
 Connection ~ 3800 3200
 Connection ~ 4550 3200
-Text Label 5950 3050 0    50   ~ 0
+Text Label 5550 3150 0    50   ~ 0
 GND1
-Text Label 5950 2300 0    50   ~ 0
+Text Label 5600 2350 0    50   ~ 0
 GND1
-Wire Wire Line
-	6150 1900 6850 1900
-Wire Wire Line
-	6850 1900 6850 2750
-Wire Wire Line
-	6850 2750 7100 2750
-Wire Wire Line
-	6150 2650 6750 2650
-Wire Wire Line
-	6750 2650 6750 2750
-Wire Wire Line
-	6750 2750 6850 2750
-Connection ~ 6850 2750
-Wire Wire Line
-	6150 2000 6550 2000
-Wire Wire Line
-	6550 2000 6550 2850
-Wire Wire Line
-	6550 2850 7100 2850
-Wire Wire Line
-	6150 2750 6500 2750
-Wire Wire Line
-	6500 2750 6500 2850
-Wire Wire Line
-	6500 2850 6550 2850
-Connection ~ 6550 2850
-Text Label 6150 2100 0    50   ~ 0
+Text Label 5800 2150 0    50   ~ 0
 VCC1
 Text Label 8500 2650 0    50   ~ 0
@@
 NoConn ~ 14050 1150
 NoConn ~ 12800 2250
+Text Label 6750 3700 0    50   ~ 0
+VCC1
+$Comp
+L Analog_Switch:ADG417BN U?
+U 1 1 5C9D336E
+P 6450 3700
+F 0 "U?" H 6450 3967 50  0000 C CNN
+F 1 "ADG417BN" H 6450 3876 50  0000 C CNN
+F 2 "Connector_PinHeader_2.54mm:PinHeader_1x03_P2.54mm_Vertical" H 6450 3600 50  0001 C CNN
+F 3 "http://www.analog.com/media/en/technical-documentation/data-sheets/ADG417.pdf" H 6450 3700 50  0001 C CNN
+	1    6450 3700
+	-1   0    0    1
+$EndComp
+Wire Wire Line
+	5750 2850 6100 2850
+Wire Wire Line
+	5750 2750 6250 2750
+Wire Wire Line
+	5800 2050 6100 2050
+Wire Wire Line
+	6100 2050 6100 2850
+Connection ~ 6100 2850
+Wire Wire Line
+	6100 2850 6450 2850
+Wire Wire Line
+	5800 1950 6250 1950
+Wire Wire Line
+	6250 1950 6250 2750
+Connection ~ 6250 2750
+Wire Wire Line
+	6250 2750 6700 2750
+Wire Wire Line
+	6450 3500 6700 3500
+Wire Wire Line
+	6700 3500 6700 3300
+$Comp
+L Device:R R?
+U 1 1 5C9F1D14
+P 6700 3150
+F 0 "R?" H 6770 3196 50  0000 L CNN
+F 1 "R" H 6770 3105 50  0000 L CNN
+F 2 "" V 6630 3150 50  0001 C CNN
+F 3 "~" H 6700 3150 50  0001 C CNN
+	1    6700 3150
+	1    0    0    -1
+$EndComp
+$Comp
+L Device:R R?
+U 1 1 5C9F1DDC
+P 6450 3150
+F 0 "R?" H 6520 3196 50  0000 L CNN
+F 1 "R" H 6520 3105 50  0000 L CNN
+F 2 "" V 6380 3150 50  0001 C CNN
+F 3 "~" H 6450 3150 50  0001 C CNN
+	1    6450 3150
+	1    0    0    -1
+$EndComp
+Wire Wire Line
+	6450 3500 6450 3300
+Connection ~ 6450 3500
+Wire Wire Line
+	6450 3000 6450 2850
+Connection ~ 6450 2850
+Wire Wire Line
+	6450 2850 7100 2850
+Wire Wire Line
+	6700 3000 6700 2750
+Connection ~ 6700 2750
+Wire Wire Line
+	6700 2750 7100 2750
 $EndSCHEMATC

Commit message: layed out components
Parts:
- added U6: ADG417BN, Connector_PinHeader_2.54mm:PinHeader_1x03_P2.54mm_Vertical, symbol Analog_Switch:ADG417BN
- R1, R2: renamed from R?; footprint (none) -> keyboard_parts:D_SOD123_axial
- U1: footprint promicro:ProMicro -> foots:ProMicroPinsFlipped
- gave numbers to parts that had none: 1
Changed lines of the file:
@@
 F 0 "U1" H 7800 4137 60  0000 C CNN
 F 1 "ProMicro" H 7800 4031 60  0000 C CNN
-F 2 "promicro:ProMicro" H 7900 2050 60  0001 C CNN
+F 2 "foots:ProMicroPinsFlipped" H 7900 2050 60  0001 C CNN
 F 3 "" H 7900 2050 60  0000 C CNN
 	1    7800 3100
@@
 Text Label 8500 2650 0    50   ~ 0
 VCC1
-Text Label 9600 2100 2    50   ~ 0
+Text Label 9300 2300 0    50   ~ 0
 VCC1
 NoConn ~ 7100 2450
@@
 VCC1
 $Comp
-L Analog_Switch:ADG417BN U?
+L Analog_Switch:ADG417BN U5
 U 1 1 5C9D336E
 P 6450 3700
-F 0 "U?" H 6450 3967 50  0000 C CNN
+F 0 "U5" H 6450 3967 50  0000 C CNN
 F 1 "ADG417BN" H 6450 3876 50  0000 C CNN
 F 2 "Connector_PinHeader_2.54mm:PinHeader_1x03_P2.54mm_Vertical" H 6450 3600 50  0001 C CNN
@@
 	6700 3500 6700 3300
 $Comp
-L Device:R R?
+L Device:R R2
 U 1 1 5C9F1D14
 P 6700 3150
-F 0 "R?" H 6770 3196 50  0000 L CNN
+F 0 "R2" H 6770 3196 50  0000 L CNN
 F 1 "R" H 6770 3105 50  0000 L CNN
-F 2 "" V 6630 3150 50  0001 C CNN
+F 2 "keyboard_parts:D_SOD123_axial" V 6630 3150 50  0001 C CNN
 F 3 "~" H 6700 3150 50  0001 C CNN
 	1    6700 3150
@@
 $EndComp
 $Comp
-L Device:R R?
+L Device:R R1
 U 1 1 5C9F1DDC
 P 6450 3150
-F 0 "R?" H 6520 3196 50  0000 L CNN
+F 0 "R1" H 6520 3196 50  0000 L CNN
 F 1 "R" H 6520 3105 50  0000 L CNN
-F 2 "" V 6380 3150 50  0001 C CNN
+F 2 "keyboard_parts:D_SOD123_axial" V 6380 3150 50  0001 C CNN
 F 3 "~" H 6450 3150 50  0001 C CNN
 	1    6450 3150
@@
 Wire Wire Line
 	6700 2750 7100 2750
+$Comp
+L Analog_Switch:ADG417BN U6
+U 1 1 5CA64439
+P 9300 2100
+F 0 "U6" H 9300 2367 50  0000 C CNN
+F 1 "ADG417BN" H 9300 2276 50  0000 C CNN
+F 2 "Connector_PinHeader_2.54mm:PinHeader_1x03_P2.54mm_Vertical" H 9300 2000 50  0001 C CNN
+F 3 "http://www.analog.com/media/en/technical-documentation/data-sheets/ADG417.pdf" H 9300 2100 50  0001 C CNN
+	1    9300 2100
+	1    0    0    -1
+$EndComp
 $EndSCHEMATC

Commit message: start tracing
Parts:
- J1, J2: footprint foots:CUI_SJ1-3514-SMT[PAD1,2,34] -> foots:CUI_SJ1-3514-SMT[PAD1,2,34]Backside
Changed lines of the file:
@@
 F 0 "J1" H 5580 2375 50  0000 C CNN
 F 1 "AudioJack3_Ground" H 5580 2284 50  0000 C CNN
-F 2 "foots:CUI_SJ1-3514-SMT[PAD1,2,34]" H 5600 2050 50  0001 C CNN
+F 2 "foots:CUI_SJ1-3514-SMT[PAD1,2,34]Backside" H 5600 2050 50  0001 C CNN
 F 3 "~" H 5600 2050 50  0001 C CNN
 	1    5600 2050
@@
 F 0 "J2" H 5530 3175 50  0000 C CNN
 F 1 "AudioJack3_Ground" H 5530 3084 50  0000 C CNN
-F 2 "foots:CUI_SJ1-3514-SMT[PAD1,2,34]" H 5550 2850 50  0001 C CNN
+F 2 "foots:CUI_SJ1-3514-SMT[PAD1,2,34]Backside" H 5550 2850 50  0001 C CNN
 F 3 "~" H 5550 2850 50  0001 C CNN
 	1    5550 2850

Commit message: started led matrix
Parts:
- added D20, D21, D22, D23, D24, D25, D26, D27, D28, D29, D30, D31, D32, D33, D34, D35: LED, symbol Device:LED
- added U?: MSP430G2553IN20, Package_DIP:DIP-20_W7.62mm, symbol MCU_Texas_MSP430:MSP430G2553IN20
Connections:
- net labels added: GND2
- wire segments 68 -> 125

Commit message: TLC5940 LED controller
Parts:
- removed U?: MSP430G2553IN20, Package_DIP:DIP-20_W7.62mm, symbol MCU_Texas_MSP430:MSP430G2553IN20
- added U7: TLC5940PWP, Package_SO:HTSSOP-28-1EP_4.4x9.7mm_P0.65mm_EP3.4x9.5mm_Mask2.4x6.17mm_ThermalVias, symbol Driver_LED:TLC5940PWP
- D1: footprint keyboard_parts:D_SOD123_axial -> keyboard_parts:C_3528
- D20, D21, D22, D23, D24, D25, D26, D27, D28, D29, D30, D31, D32, D33, D34, D35: footprint (none) -> keyboard_parts:C_3528
Connections:
- net labels added: GSCLK
- net labels removed: GND2
- wire segments 125 -> 144
- no-connect marks 10 -> 7

Commit message: traces from led ic
Parts:
- D1: footprint keyboard_parts:C_3528 -> keyboard_parts:D_SOD123_axial
- J1, J2: footprint foots:CUI_SJ1-3514-SMT[PAD1,2,34]Backside -> foots:CUI_SJ-43514-SMT(1,2,3,4reverseside)
Changed lines of the file:
@@
 F 0 "D1" V 1746 1921 50  0000 R CNN
 F 1 "D" V 1655 1921 50  0000 R CNN
-F 2 "keyboard_parts:C_3528" H 1700 2000 50  0001 C CNN
+F 2 "keyboard_parts:D_SOD123_axial" H 1700 2000 50  0001 C CNN
 F 3 "~" H 1700 2000 50  0001 C CNN
 	1    1700 2000
@@
 F 0 "J1" H 5580 2375 50  0000 C CNN
 F 1 "AudioJack3_Ground" H 5580 2284 50  0000 C CNN
-F 2 "foots:CUI_SJ1-3514-SMT[PAD1,2,34]Backside" H 5600 2050 50  0001 C CNN
+F 2 "foots:CUI_SJ-43514-SMT(1,2,3,4reverseside)" H 5600 2050 50  0001 C CNN
 F 3 "~" H 5600 2050 50  0001 C CNN
 	1    5600 2050
@@
 F 0 "J2" H 5530 3175 50  0000 C CNN
 F 1 "AudioJack3_Ground" H 5530 3084 50  0000 C CNN
-F 2 "foots:CUI_SJ1-3514-SMT[PAD1,2,34]Backside" H 5550 2850 50  0001 C CNN
+F 2 "foots:CUI_SJ-43514-SMT(1,2,3,4reverseside)" H 5550 2850 50  0001 C CNN
 F 3 "~" H 5550 2850 50  0001 C CNN
 	1    5550 2850
