File: pcb_files/arrowPad.sch (KiCad schematic (older format))
At the start: 60 parts, among them J1 AudioJack3_Ground, J2 AudioJack3_Ground, K1 KEYSW, K10 KEYSW, K11 KEYSW, K12 KEYSW, K13 KEYSW, K14 KEYSW, K15 KEYSW, K16 KEYSW, K2 KEYSW, K3 KEYSW, K4 KEYSW, K5 KEYSW, K6 KEYSW, K7 KEYSW, K8 KEYSW, K9 KEYSW, U1 ProMicro, U2 NRF24L01_Breakout, U3 ADG417BN, U4 AMS1117-3.3, U5 ADG417BN, U6 ADG417BN, U7 TLC5940PWP

Commit message: adding TLC5940 connections
Parts:
- added R?: R, symbol Device:R
- D20, D21, D22, D23, D24, D25, D26, D27, D28, D29, D30, D31, D32, D33, D34, D35: footprint keyboard_parts:C_3528 -> foots:C_3528v1
- J1, J2: footprint foots:CUI_SJ-43514-SMT(1,2,3,4reverseside) -> SJ-43514-SMT:CUI_SJ-43514-SMT
Connections:
- wire segments 144 -> 149
Changed lines of the file:
@@
 F 0 "J1" H 5580 2375 50  0000 C CNN
 F 1 "AudioJack3_Ground" H 5580 2284 50  0000 C CNN
-F 2 "foots:CUI_SJ-43514-SMT(1,2,3,4reverseside)" H 5600 2050 50  0001 C CNN
+F 2 "SJ-43514-SMT:CUI_SJ-43514-SMT" H 5600 2050 50  0001 C CNN
 F 3 "~" H 5600 2050 50  0001 C CNN
 	1    5600 2050
@@
 F 0 "J2" H 5530 3175 50  0000 C CNN
 F 1 "AudioJack3_Ground" H 5530 3084 50  0000 C CNN
-F 2 "foots:CUI_SJ-43514-SMT(1,2,3,4reverseside)" H 5550 2850 50  0001 C CNN
+F 2 "SJ-43514-SMT:CUI_SJ-43514-SMT" H 5550 2850 50  0001 C CNN
 F 3 "~" H 5550 2850 50  0001 C CNN
 	1    5550 2850
@@
 F 0 "D20" V 6845 5079 50  0000 L CNN
 F 1 "LED" V 6936 5079 50  0000 L CNN
-F 2 "keyboard_parts:C_3528" H 6900 5000 50  0001 C CNN
+F 2 "foots:C_3528v1" H 6900 5000 50  0001 C CNN
 F 3 "~" H 6900 5000 50  0001 C CNN
 	1    6900 5000
@@
 F 0 "D21" V 6545 5079 50  0000 L CNN
 F 1 "LED" V 6636 5079 50  0000 L CNN
-F 2 "keyboard_parts:C_3528" H 6600 5000 50  0001 C CNN
+F 2 "foots:C_3528v1" H 6600 5000 50  0001 C CNN
 F 3 "~" H 6600 5000 50  0001 C CNN
 	1    6600 5000
@@
 F 0 "D22" V 6245 5079 50  0000 L CNN
 F 1 "LED" V 6336 5079 50  0000 L CNN
-F 2 "keyboard_parts:C_3528" H 6300 5000 50  0001 C CNN
+F 2 "foots:C_3528v1" H 6300 5000 50  0001 C CNN
 F 3 "~" H 6300 5000 50  0001 C CNN
 	1    6300 5000
@@
 F 0 "D23" V 5945 5079 50  0000 L CNN
 F 1 "LED" V 6036 5079 50  0000 L CNN
-F 2 "keyboard_parts:C_3528" H 6000 5000 50  0001 C CNN
+F 2 "foots:C_3528v1" H 6000 5000 50  0001 C CNN
 F 3 "~" H 6000 5000 50  0001 C CNN
 	1    6000 5000
@@
 F 0 "D24" V 5645 5079 50  0000 L CNN
 F 1 "LED" V 5736 5079 50  0000 L CNN
-F 2 "keyboard_parts:C_3528" H 5700 5000 50  0001 C CNN
+F 2 "foots:C_3528v1" H 5700 5000 50  0001 C CNN
 F 3 "~" H 5700 5000 50  0001 C CNN
 	1    5700 5000
@@
 F 0 "D25" V 5345 5079 50  0000 L CNN
 F 1 "LED" V 5436 5079 50  0000 L CNN
-F 2 "keyboard_parts:C_3528" H 5400 5000 50  0001 C CNN
+F 2 "foots:C_3528v1" H 5400 5000 50  0001 C CNN
 F 3 "~" H 5400 5000 50  0001 C CNN
 	1    5400 5000
@@
 F 0 "D26" V 5045 5079 50  0000 L CNN
 F 1 "LED" V 5136 5079 50  0000 L CNN
-F 2 "keyboard_parts:C_3528" H 5100 5000 50  0001 C CNN
+F 2 "foots:C_3528v1" H 5100 5000 50  0001 C CNN
 F 3 "~" H 5100 5000 50  0001 C CNN
 	1    5100 5000
@@
 F 0 "D27" V 4745 5079 50  0000 L CNN
 F 1 "LED" V 4836 5079 50  0000 L CNN
-F 2 "keyboard_parts:C_3528" H 4800 5000 50  0001 C CNN
+F 2 "foots:C_3528v1" H 4800 5000 50  0001 C CNN
 F 3 "~" H 4800 5000 50  0001 C CNN
 	1    4800 5000
@@
 F 0 "D28" V 4445 5079 50  0000 L CNN
 F 1 "LED" V 4536 5079 50  0000 L CNN
-F 2 "keyboard_parts:C_3528" H 4500 5000 50  0001 C CNN
+F 2 "foots:C_3528v1" H 4500 5000 50  0001 C CNN
 F 3 "~" H 4500 5000 50  0001 C CNN
 	1    4500 5000
@@
 F 0 "D29" V 4145 5079 50  0000 L CNN
 F 1 "LED" V 4236 5079 50  0000 L CNN
-F 2 "keyboard_parts:C_3528" H 4200 5000 50  0001 C CNN
+F 2 "foots:C_3528v1" H 4200 5000 50  0001 C CNN
 F 3 "~" H 4200 5000 50  0001 C CNN
 	1    4200 5000
@@
 F 0 "D30" V 3845 5079 50  0000 L CNN
 F 1 "LED" V 3936 5079 50  0000 L CNN
-F 2 "keyboard_parts:C_3528" H 3900 5000 50  0001 C CNN
+F 2 "foots:C_3528v1" H 3900 5000 50  0001 C CNN
 F 3 "~" H 3900 5000 50  0001 C CNN
 	1    3900 5000
@@
 F 0 "D31" V 3545 5079 50  0000 L CNN
 F 1 "LED" V 3636 5079 50  0000 L CNN
-F 2 "keyboard_parts:C_3528" H 3600 5000 50  0001 C CNN
+F 2 "foots:C_3528v1" H 3600 5000 50  0001 C CNN
 F 3 "~" H 3600 5000 50  0001 C CNN
 	1    3600 5000
@@
 F 0 "D32" V 3245 5079 50  0000 L CNN
 F 1 "LED" V 3336 5079 50  0000 L CNN
-F 2 "keyboard_parts:C_3528" H 3300 5000 50  0001 C CNN
+F 2 "foots:C_3528v1" H 3300 5000 50  0001 C CNN
 F 3 "~" H 3300 5000 50  0001 C CNN
 	1    3300 5000
@@
 F 0 "D33" V 2945 5079 50  0000 L CNN
 F 1 "LED" V 3036 5079 50  0000 L CNN
-F 2 "keyboard_parts:C_3528" H 3000 5000 50  0001 C CNN
+F 2 "foots:C_3528v1" H 3000 5000 50  0001 C CNN
 F 3 "~" H 3000 5000 50  0001 C CNN
 	1    3000 5000
@@
 F 0 "D34" V 2645 5079 50  0000 L CNN
 F 1 "LED" V 2736 5079 50  0000 L CNN
-F 2 "keyboard_parts:C_3528" H 2700 5000 50  0001 C CNN
+F 2 "foots:C_3528v1" H 2700 5000 50  0001 C CNN
 F 3 "~" H 2700 5000 50  0001 C CNN
 	1    2700 5000
@@
 F 0 "D35" V 2345 5079 50  0000 L CNN
 F 1 "LED" V 2436 5079 50  0000 L CNN
-F 2 "keyboard_parts:C_3528" H 2400 5000 50  0001 C CNN
+F 2 "foots:C_3528v1" H 2400 5000 50  0001 C CNN
 F 3 "~" H 2400 5000 50  0001 C CNN
 	1    2400 5000
@@
 Text Label 2000 4850 2    50   ~ 0
 GND1
+Wire Wire Line
+	8950 3900 8950 3700
+Wire Wire Line
+	8850 3700 8850 3900
+$Comp
+L Device:R R?
+U 1 1 5CC8653E
+P 8850 3550
+F 0 "R?" H 8920 3596 50  0000 L CNN
+F 1 "R" H 8920 3505 50  0000 L CNN
+F 2 "" V 8780 3550 50  0001 C CNN
+F 3 "~" H 8850 3550 50  0001 C CNN
+	1    8850 3550
+	1    0    0    -1
+$EndComp
+Wire Wire Line
+	8750 3900 8750 3700
+Wire Wire Line
+	9250 4600 9550 4600
+Wire Wire Line
+	9550 4600 9550 4300
 $EndSCHEMATC

Commit message: cleaned up board text
Parts:
- R3: renamed from R?; footprint (none) -> keyboard_parts:D_SOD123_axial
Connections:
- wire segments 149 -> 148
Changed lines of the file:
@@
 Wire Wire Line
 	6600 4850 6900 4850
-Text Label 2000 4850 2    50   ~ 0
-GND1
-Wire Wire Line
-	8950 3900 8950 3700
 Wire Wire Line
 	8850 3700 8850 3900
 $Comp
-L Device:R R?
+L Device:R R3
 U 1 1 5CC8653E
-P 8850 3550
-F 0 "R?" H 8920 3596 50  0000 L CNN
-F 1 "R" H 8920 3505 50  0000 L CNN
-F 2 "" V 8780 3550 50  0001 C CNN
-F 3 "~" H 8850 3550 50  0001 C CNN
-	1    8850 3550
-	1    0    0    -1
+P 9000 3700
+F 0 "R3" V 8793 3700 50  0000 C CNN
+F 1 "R" V 8884 3700 50  0000 C CNN
+F 2 "keyboard_parts:D_SOD123_axial" V 8930 3700 50  0001 C CNN
+F 3 "~" H 9000 3700 50  0001 C CNN
+	1    9000 3700
+	0    1    1    0
 $EndComp
 Wire Wire Line
@@
 Wire Wire Line
 	9550 4600 9550 4300
+Text Label 8950 3900 0    50   ~ 0
+GND1
+Text Label 8850 3400 0    50   ~ 0
+GND1
+Text Label 9150 3700 0    50   ~ 0
+GND1
+Text Label 2000 4850 0    50   ~ 0
+VCC1
+Text Label 9550 4300 0    50   ~ 0
+VCC1
+Text Label 8750 3700 1    50   ~ 0
+VCC1
 $EndSCHEMATC

Commit message: added image for pcb
Parts:
- U4: footprint promicro:AMS1117flipped -> AMS1117-3.3:SOT229P700X180-4N
Connections:
- no-connect marks 7 -> 6
Changed lines of the file:
@@
 F 0 "U4" H 10200 2567 50  0000 C CNN
 F 1 "AMS1117-3.3" H 10200 2476 50  0000 C CNN
-F 2 "promicro:AMS1117flipped" H 10200 2200 50  0001 L BNN
+F 2 "AMS1117-3.3:SOT229P700X180-4N" H 10200 2200 50  0001 L BNN
 F 3 "Sot223/Pkg 1-Amp 3.3-Volt Low Drop Out Voltage Regulatator" H 10200 2200 50  0001 L BNN
 F 4 "Advanced Monolithic Systems" H 10200 2200 50  0001 L BNN "Field4"
@@
 NoConn ~ 7900 1250
 NoConn ~ 14050 1150
-NoConn ~ 12800 2250
 Text Label 6750 3700 0    50   ~ 0
 VCC1
@@
 Text Label 2000 4850 0    50   ~ 0
 VCC1
+Text Label 8750 3700 1    50   ~ 0
+VCC1
 Text Label 9550 4300 0    50   ~ 0
 VCC1
-Text Label 8750 3700 1    50   ~ 0
-VCC1
 $EndSCHEMATC
