File: pcb_files/arrowPad.sch (KiCad schematic (older format))
At the start: 61 parts, among them J1 AudioJack3_Ground, J2 AudioJack3_Ground, K1 KEYSW, K10 KEYSW, K11 KEYSW, K12 KEYSW, K13 KEYSW, K14 KEYSW, K15 KEYSW, K16 KEYSW, K2 KEYSW, K3 KEYSW, K4 KEYSW, K5 KEYSW, K6 KEYSW, K7 KEYSW, K8 KEYSW, K9 KEYSW, U1 ProMicro, U2 NRF24L01_Breakout, U3 ADG417BN, U4 AMS1117-3.3, U5 ADG417BN, U6 ADG417BN, U7 TLC5940PWP

Commit message: re added mounting holes
Parts:
- D1, D10, D11, D12, D13, D14, D15, D16, D2, D3, D4, D5, D6, D7, D8, D9: footprint keyboard_parts:D_SOD123_axial -> keyboard_parts:D_SOD123_axial_noSMD
Changed lines of the file:
@@
 F 0 "D3" V 3250 1900 50  0000 C CNN
 F 1 "D" V 3150 1900 50  0000 C CNN
-F 2 "keyboard_parts:D_SOD123_axial" H 3200 2000 50  0001 C CNN
+F 2 "keyboard_parts:D_SOD123_axial_noSMD" H 3200 2000 50  0001 C CNN
 F 3 "~" H 3200 2000 50  0001 C CNN
 	1    3200 2000
@@
 F 0 "D2" V 2496 1921 50  0000 R CNN
 F 1 "D" V 2405 1921 50  0000 R CNN
-F 2 "keyboard_parts:D_SOD123_axial" H 2450 2000 50  0001 C CNN
+F 2 "keyboard_parts:D_SOD123_axial_noSMD" H 2450 2000 50  0001 C CNN
 F 3 "~" H 2450 2000 50  0001 C CNN
 	1    2450 2000
@@
 F 0 "D1" V 1746 1921 50  0000 R CNN
 F 1 "D" V 1655 1921 50  0000 R CNN
-F 2 "keyboard_parts:D_SOD123_axial" H 1700 2000 50  0001 C CNN
+F 2 "keyboard_parts:D_SOD123_axial_noSMD" H 1700 2000 50  0001 C CNN
 F 3 "~" H 1700 2000 50  0001 C CNN
 	1    1700 2000
@@
 F 0 "D5" V 1746 2571 50  0000 R CNN
 F 1 "D" V 1655 2571 50  0000 R CNN
-F 2 "keyboard_parts:D_SOD123_axial" H 1700 2650 50  0001 C CNN
+F 2 "keyboard_parts:D_SOD123_axial_noSMD" H 1700 2650 50  0001 C CNN
 F 3 "~" H 1700 2650 50  0001 C CNN
 	1    1700 2650
@@
 F 0 "D6" V 2496 2571 50  0000 R CNN
 F 1 "D" V 2405 2571 50  0000 R CNN
-F 2 "keyboard_parts:D_SOD123_axial" H 2450 2650 50  0001 C CNN
+F 2 "keyboard_parts:D_SOD123_axial_noSMD" H 2450 2650 50  0001 C CNN
 F 3 "~" H 2450 2650 50  0001 C CNN
 	1    2450 2650
@@
 F 0 "D7" V 3246 2571 50  0000 R CNN
 F 1 "D" V 3155 2571 50  0000 R CNN
-F 2 "keyboard_parts:D_SOD123_axial" H 3200 2650 50  0001 C CNN
+F 2 "keyboard_parts:D_SOD123_axial_noSMD" H 3200 2650 50  0001 C CNN
 F 3 "~" H 3200 2650 50  0001 C CNN
 	1    3200 2650
@@
 F 0 "D9" V 1746 3271 50  0000 R CNN
 F 1 "D" V 1655 3271 50  0000 R CNN
-F 2 "keyboard_parts:D_SOD123_axial" H 1700 3350 50  0001 C CNN
+F 2 "keyboard_parts:D_SOD123_axial_noSMD" H 1700 3350 50  0001 C CNN
 F 3 "~" H 1700 3350 50  0001 C CNN
 	1    1700 3350
@@
 F 0 "D10" V 2496 3271 50  0000 R CNN
 F 1 "D" V 2405 3271 50  0000 R CNN
-F 2 "keyboard_parts:D_SOD123_axial" H 2450 3350 50  0001 C CNN
+F 2 "keyboard_parts:D_SOD123_axial_noSMD" H 2450 3350 50  0001 C CNN
 F 3 "~" H 2450 3350 50  0001 C CNN
 	1    2450 3350
@@
 F 0 "D11" V 3246 3271 50  0000 R CNN
 F 1 "D" V 3155 3271 50  0000 R CNN
-F 2 "keyboard_parts:D_SOD123_axial" H 3200 3350 50  0001 C CNN
+F 2 "keyboard_parts:D_SOD123_axial_noSMD" H 3200 3350 50  0001 C CNN
 F 3 "~" H 3200 3350 50  0001 C CNN
 	1    3200 3350
@@
 F 0 "D4" V 4000 1900 50  0000 C CNN
 F 1 "D" V 3900 1900 50  0000 C CNN
-F 2 "keyboard_parts:D_SOD123_axial" H 3950 2000 50  0001 C CNN
+F 2 "keyboard_parts:D_SOD123_axial_noSMD" H 3950 2000 50  0001 C CNN
 F 3 "~" H 3950 2000 50  0001 C CNN
 	1    3950 2000
@@
 F 0 "D8" V 3996 2571 50  0000 R CNN
 F 1 "D" V 3905 2571 50  0000 R CNN
-F 2 "keyboard_parts:D_SOD123_axial" H 3950 2650 50  0001 C CNN
+F 2 "keyboard_parts:D_SOD123_axial_noSMD" H 3950 2650 50  0001 C CNN
 F 3 "~" H 3950 2650 50  0001 C CNN
 	1    3950 2650
@@
 F 0 "D12" V 3996 3271 50  0000 R CNN
 F 1 "D" V 3905 3271 50  0000 R CNN
-F 2 "keyboard_parts:D_SOD123_axial" H 3950 3350 50  0001 C CNN
+F 2 "keyboard_parts:D_SOD123_axial_noSMD" H 3950 3350 50  0001 C CNN
 F 3 "~" H 3950 3350 50  0001 C CNN
 	1    3950 3350
@@
 F 0 "D13" V 1746 3971 50  0000 R CNN
 F 1 "D" V 1655 3971 50  0000 R CNN
-F 2 "keyboard_parts:D_SOD123_axial" H 1700 4050 50  0001 C CNN
+F 2 "keyboard_parts:D_SOD123_axial_noSMD" H 1700 4050 50  0001 C CNN
 F 3 "~" H 1700 4050 50  0001 C CNN
 	1    1700 4050
@@
 F 0 "D14" V 2496 3971 50  0000 R CNN
 F 1 "D" V 2405 3971 50  0000 R CNN
-F 2 "keyboard_parts:D_SOD123_axial" H 2450 4050 50  0001 C CNN
+F 2 "keyboard_parts:D_SOD123_axial_noSMD" H 2450 4050 50  0001 C CNN
 F 3 "~" H 2450 4050 50  0001 C CNN
 	1    2450 4050
@@
 F 0 "D15" V 3246 3971 50  0000 R CNN
 F 1 "D" V 3155 3971 50  0000 R CNN
-F 2 "keyboard_parts:D_SOD123_axial" H 3200 4050 50  0001 C CNN
+F 2 "keyboard_parts:D_SOD123_axial_noSMD" H 3200 4050 50  0001 C CNN
 F 3 "~" H 3200 4050 50  0001 C CNN
 	1    3200 4050
@@
 F 0 "D16" V 3996 3971 50  0000 R CNN
 F 1 "D" V 3905 3971 50  0000 R CNN
-F 2 "keyboard_parts:D_SOD123_axial" H 3950 4050 50  0001 C CNN
+F 2 "keyboard_parts:D_SOD123_axial_noSMD" H 3950 4050 50  0001 C CNN
 F 3 "~" H 3950 4050 50  0001 C CNN
 	1    3950 4050
