File: receiver/receiver.kicad_pcb (KiCad board)
At the start: 2 copper layers, 32.7 x 20 mm, 4 parts, among them U1 ProMicro, U2 NRF24L01_Breakout, U3 NRF24L01_Breakout, U4 AMS1117-3.3

Commit message: pcb sent to print
Parts:
- moved U4 3.52 mm to (145.7, 84.3), turned to 90 degrees
Routing:
- net /VCC1: track 36.9 -> 46.8 mm
- net /3.3V: track 15.6 -> 16.6 mm
Other:
- board size 32.7 x 20 mm -> 34.5 x 20 mm
