File: pcbV2/_autosave-keypadV2.sch (KiCad schematic (older format))
At the start: 72 parts

Commit message: start mapping symbols and footprints
Parts:
- C1, C10, C11, C12, C13, C14, C15, C16, C2, C3, C4, C5, C6, C7, C8, C9: renamed from C?; footprint (none) -> Capacitor_SMD:C_1206_3216Metric_Pad1.42x1.75mm_HandSolder
- D1, D10, D11, D12, D2, D3, D4, D5, D6, D7, D8, D9: renamed from D?; footprint (none) -> Diode_SMD:D_SOD-323_HandSoldering
- gave numbers to parts that had none: 44
Other:
- moved on the sheet: D13, R1, SW13, SW14

Commit message: save
Parts:
- D13: footprint (none) -> LED_SMD:LED_1206_3216Metric_Pad1.42x1.75mm_HandSolder
- J1: footprint (none) -> Connector_PinHeader_2.00mm:PinHeader_1x02_P2.00mm_Vertical
- Q1: footprint (none) -> Package_TO_SOT_SMD:SOT-23
- R1, R2, R3, R4, R5: footprint (none) -> Resistor_SMD:R_1206_3216Metric_Pad1.42x1.75mm_HandSolder
- SW1, SW10, SW11, SW12, SW2, SW3, SW4, SW5, SW6, SW7, SW8, SW9: footprint (none) -> keyswitches:Kailh_socket_MX
- SW13: footprint (none) -> Connector_PinHeader_2.54mm:PinHeader_1x03_P2.54mm_Vertical
- U2: footprint (none) -> Connector_PinHeader_2.54mm:PinHeader_1x07_P2.54mm_Vertical
Changed lines of the file:
@@
 F 0 "D13" H 14943 7445 50  0000 C CNN
 F 1 "LED" H 14943 7536 50  0000 C CNN
-F 2 "" H 14950 7700 50  0001 C CNN
+F 2 "LED_SMD:LED_1206_3216Metric_Pad1.42x1.75mm_HandSolder" H 14950 7700 50  0001 C CNN
 F 3 "~" H 14950 7700 50  0001 C CNN
 	1    14950 7700
@@
 F 0 "SW13" H 14800 6785 50  0000 C CNN
 F 1 "SW_SPDT" H 14800 6694 50  0000 C CNN
-F 2 "" H 14800 6500 50  0001 C CNN
+F 2 "Connector_PinHeader_2.54mm:PinHeader_1x03_P2.54mm_Vertical" H 14800 6500 50  0001 C CNN
 F 3 "~" H 14800 6500 50  0001 C CNN
 	1    14800 6500
@@
 F 0 "SW1" H 16350 3335 50  0000 C CNN
 F 1 "SW_Push" H 16350 3244 50  0000 C CNN
-F 2 "" H 16350 3250 50  0001 C CNN
+F 2 "keyswitches:Kailh_socket_MX" H 16350 3250 50  0001 C CNN
 F 3 "~" H 16350 3250 50  0001 C CNN
 	1    16350 3050
@@
 F 0 "R2" H 6270 9246 50  0000 L CNN
 F 1 "10K" H 6270 9155 50  0000 L CNN
-F 2 "" V 6130 9200 50  0001 C CNN
+F 2 "Resistor_SMD:R_1206_3216Metric_Pad1.42x1.75mm_HandSolder" V 6130 9200 50  0001 C CNN
 F 3 "~" H 6200 9200 50  0001 C CNN
 	1    6200 9200
@@
 F 0 "U2" H 4008 7065 50  0000 C CNN
 F 1 "Waveshare_OLED_RGB" H 4008 6974 50  0000 C CNN
-F 2 "" H 4150 5400 50  0001 C CNN
+F 2 "Connector_PinHeader_2.54mm:PinHeader_1x07_P2.54mm_Vertical" H 4150 5400 50  0001 C CNN
 F 3 "" H 4150 5400 50  0001 C CNN
 	1    3950 5400
@@
 F 0 "R4" V 19193 9600 50  0000 C CNN
 F 1 "0" V 19284 9600 50  0000 C CNN
-F 2 "" V 19330 9600 50  0001 C CNN
+F 2 "Resistor_SMD:R_1206_3216Metric_Pad1.42x1.75mm_HandSolder" V 19330 9600 50  0001 C CNN
 F 3 "~" H 19400 9600 50  0001 C CNN
 	1    19400 9600
@@
 F 0 "R1" V 14707 7700 50  0000 C CNN
 F 1 "R" V 14616 7700 50  0000 C CNN
-F 2 "" V 14430 7700 50  0001 C CNN
+F 2 "Resistor_SMD:R_1206_3216Metric_Pad1.42x1.75mm_HandSolder" V 14430 7700 50  0001 C CNN
 F 3 "~" H 14500 7700 50  0001 C CNN
 	1    14500 7700
@@
 F 0 "Q1" V 6849 9350 50  0000 C CNN
 F 1 "Q_NMOS_GSD" V 6940 9350 50  0000 C CNN
-F 2 "" H 6800 9450 50  0001 C CNN
+F 2 "Package_TO_SOT_SMD:SOT-23" H 6800 9450 50  0001 C CNN
 F 3 "~" H 6600 9350 50  0001 C CNN
 	1    6600 9350
@@
 F 0 "R3" H 7120 9246 50  0000 L CNN
 F 1 "10K" H 7120 9155 50  0000 L CNN
-F 2 "" V 6980 9200 50  0001 C CNN
+F 2 "Resistor_SMD:R_1206_3216Metric_Pad1.42x1.75mm_HandSolder" V 6980 9200 50  0001 C CNN
 F 3 "~" H 7050 9200 50  0001 C CNN
 	1    7050 9200
@@
 F 0 "R5" V 5893 10000 50  0000 C CNN
 F 1 "R" V 5984 10000 50  0000 C CNN
-F 2 "" V 6030 10000 50  0001 C CNN
+F 2 "Resistor_SMD:R_1206_3216Metric_Pad1.42x1.75mm_HandSolder" V 6030 10000 50  0001 C CNN
 F 3 "~" H 6100 10000 50  0001 C CNN
 	1    6100 10000
@@
 F 0 "J1" H 18578 7876 50  0000 L CNN
 F 1 "Conn_01x02_Female" H 18578 7785 50  0000 L CNN
-F 2 "" H 18550 7900 50  0001 C CNN
+F 2 "Connector_PinHeader_2.00mm:PinHeader_1x02_P2.00mm_Vertical" H 18550 7900 50  0001 C CNN
 F 3 "~" H 18550 7900 50  0001 C CNN
 	1    18550 7900
@@
 F 0 "SW2" H 17450 3335 50  0000 C CNN
 F 1 "SW_Push" H 17450 3244 50  0000 C CNN
-F 2 "" H 17450 3250 50  0001 C CNN
+F 2 "keyswitches:Kailh_socket_MX" H 17450 3250 50  0001 C CNN
 F 3 "~" H 17450 3250 50  0001 C CNN
 	1    17450 3050
@@
 F 0 "SW3" H 18550 3335 50  0000 C CNN
 F 1 "SW_Push" H 18550 3244 50  0000 C CNN
-F 2 "" H 18550 3250 50  0001 C CNN
+F 2 "keyswitches:Kailh_socket_MX" H 18550 3250 50  0001 C CNN
 F 3 "~" H 18550 3250 50  0001 C CNN
 	1    18550 3050
@@
 F 0 "SW4" H 19650 3335 50  0000 C CNN
 F 1 "SW_Push" H 19650 3244 50  0000 C CNN
-F 2 "" H 19650 3250 50  0001 C CNN
+F 2 "keyswitches:Kailh_socket_MX" H 19650 3250 50  0001 C CNN
 F 3 "~" H 19650 3250 50  0001 C CNN
 	1    19650 3050
@@
 F 0 "SW5" H 16350 4135 50  0000 C CNN
 F 1 "SW_Push" H 16350 4044 50  0000 C CNN
-F 2 "" H 16350 4050 50  0001 C CNN
+F 2 "keyswitches:Kailh_socket_MX" H 16350 4050 50  0001 C CNN
 F 3 "~" H 16350 4050 50  0001 C CNN
 	1    16350 3850
@@
 F 0 "SW6" H 17450 4135 50  0000 C CNN
 F 1 "SW_Push" H 17450 4044 50  0000 C CNN
-F 2 "" H 17450 4050 50  0001 C CNN
+F 2 "keyswitches:Kailh_socket_MX" H 17450 4050 50  0001 C CNN
 F 3 "~" H 17450 4050 50  0001 C CNN
 	1    17450 3850
@@
 F 0 "SW7" H 18550 4135 50  0000 C CNN
 F 1 "SW_Push" H 18550 4044 50  0000 C CNN
-F 2 "" H 18550 4050 50  0001 C CNN
+F 2 "keyswitches:Kailh_socket_MX" H 18550 4050 50  0001 C CNN
 F 3 "~" H 18550 4050 50  0001 C CNN
 	1    18550 3850
@@
 F 0 "SW8" H 19650 4135 50  0000 C CNN
 F 1 "SW_Push" H 19650 4044 50  0000 C CNN
-F 2 "" H 19650 4050 50  0001 C CNN
+F 2 "keyswitches:Kailh_socket_MX" H 19650 4050 50  0001 C CNN
 F 3 "~" H 19650 4050 50  0001 C CNN
 	1    19650 3850
@@
 F 0 "SW9" H 16350 4935 50  0000 C CNN
 F 1 "SW_Push" H 16350 4844 50  0000 C CNN
-F 2 "" H 16350 4850 50  0001 C CNN
+F 2 "keyswitches:Kailh_socket_MX" H 16350 4850 50  0001 C CNN
 F 3 "~" H 16350 4850 50  0001 C CNN
 	1    16350 4650
@@
 F 0 "SW10" H 17450 4935 50  0000 C CNN
 F 1 "SW_Push" H 17450 4844 50  0000 C CNN
-F 2 "" H 17450 4850 50  0001 C CNN
+F 2 "keyswitches:Kailh_socket_MX" H 17450 4850 50  0001 C CNN
 F 3 "~" H 17450 4850 50  0001 C CNN
 	1    17450 4650
@@
 F 0 "SW11" H 18550 4935 50  0000 C CNN
 F 1 "SW_Push" H 18550 4844 50  0000 C CNN
-F 2 "" H 18550 4850 50  0001 C CNN
+F 2 "keyswitches:Kailh_socket_MX" H 18550 4850 50  0001 C CNN
 F 3 "~" H 18550 4850 50  0001 C CNN
 	1    18550 4650
@@
 F 0 "SW12" H 19650 4935 50  0000 C CNN
 F 1 "SW_Push" H 19650 4844 50  0000 C CNN
-F 2 "" H 19650 4850 50  0001 C CNN
+F 2 "keyswitches:Kailh_socket_MX" H 19650 4850 50  0001 C CNN
 F 3 "~" H 19650 4850 50  0001 C CNN
 	1    19650 4650

Commit message: start pcb layout
Parts:
- added J3: Conn_01x03_Male, Connector_PinHeader_2.00mm:PinHeader_1x03_P2.00mm_Vertical, symbol Connector:Conn_01x03_Male
- J2: footprint (none) -> custom:USB_C_REDUCED_UJ31-CH-G2
- R4: value 0 -> R_SHIELD
- R5: value R -> R_DIN
- SW14, SW15, SW16: footprint (none) -> custom:BTN_B3S-1000P
- SW17: footprint (none) -> custom:DIP3_219-3MSTR
- U1: footprint (none) -> teensy:Teensy40
Connections:
- net +5V: now also J3.1 (Pin_1)
- net GND: now also J3.3 (Pin_3)
- new net RGB_DIN: J3.2 (Pin_2)
- no-connect marks 43 -> 45
Changed lines of the file:
@@
 F 0 "U1" H 10950 6265 50  0000 C CNN
 F 1 "Teensy4.0" H 10950 6174 50  0000 C CNN
-F 2 "" H 10550 4850 50  0001 C CNN
+F 2 "teensy:Teensy40" H 10550 4850 50  0001 C CNN
 F 3 "" H 10550 4850 50  0001 C CNN
 	1    10950 4650
@@
 F 0 "SW14" H 14800 7435 50  0000 C CNN
 F 1 "SW_Push" H 14800 7344 50  0000 C CNN
-F 2 "" H 14800 7350 50  0001 C CNN
+F 2 "custom:BTN_B3S-1000P" H 14800 7350 50  0001 C CNN
 F 3 "~" H 14800 7350 50  0001 C CNN
 	1    14800 7150
@@
 F 0 "SW15" H 14450 13085 50  0000 C CNN
 F 1 "SW_Push" H 14450 12994 50  0000 C CNN
-F 2 "" H 14450 13000 50  0001 C CNN
+F 2 "custom:BTN_B3S-1000P" H 14450 13000 50  0001 C CNN
 F 3 "~" H 14450 13000 50  0001 C CNN
 	1    14450 12800
@@
 F 0 "SW16" H 14450 13585 50  0000 C CNN
 F 1 "SW_Push" H 14450 13494 50  0000 C CNN
-F 2 "" H 14450 13500 50  0001 C CNN
+F 2 "custom:BTN_B3S-1000P" H 14450 13500 50  0001 C CNN
 F 3 "~" H 14450 13500 50  0001 C CNN
 	1    14450 13300
@@
 F 0 "J2" H 18220 11197 50  0000 R CNN
 F 1 "USB_C_Receptacle" H 18220 11288 50  0000 R CNN
-F 2 "" H 18800 11500 50  0001 C CNN
+F 2 "custom:USB_C_REDUCED_UJ31-CH-G2" H 18800 11500 50  0001 C CNN
 F 3 "https://www.usb.org/sites/default/files/documents/usb_type-c.zip" H 18800 11500 50  0001 C CNN
 	1    18650 11500
@@
 F 0 "SW17" H 14450 14467 50  0000 C CNN
 F 1 "SW_DIP_x03" H 14450 14376 50  0000 C CNN
-F 2 "" H 14450 14000 50  0001 C CNN
+F 2 "custom:DIP3_219-3MSTR" H 14450 14000 50  0001 C CNN
 F 3 "~" H 14450 14000 50  0001 C CNN
 	1    14450 14000
@@
 P 19400 9600
 F 0 "R4" V 19193 9600 50  0000 C CNN
-F 1 "0" V 19284 9600 50  0000 C CNN
+F 1 "R_SHIELD" V 19284 9600 50  0000 C CNN
 F 2 "Resistor_SMD:R_1206_3216Metric_Pad1.42x1.75mm_HandSolder" V 19330 9600 50  0001 C CNN
 F 3 "~" H 19400 9600 50  0001 C CNN
@@
 P 6100 10000
 F 0 "R5" V 5893 10000 50  0000 C CNN
-F 1 "R" V 5984 10000 50  0000 C CNN
+F 1 "R_DIN" V 5984 10000 50  0000 C CNN
 F 2 "Resistor_SMD:R_1206_3216Metric_Pad1.42x1.75mm_HandSolder" V 6030 10000 50  0001 C CNN
 F 3 "~" H 6100 10000 50  0001 C CNN
@@
 NoConn ~ 12050 4800
 NoConn ~ 12050 4900
+$Comp
+L Connector:Conn_01x03_Male J3
+U 1 1 5EF9A1C0
+P 9350 9250
+F 0 "J3" H 9458 9531 50  0000 C CNN
+F 1 "Conn_01x03_Male" H 9458 9440 50  0000 C CNN
+F 2 "Connector_PinHeader_2.00mm:PinHeader_1x03_P2.00mm_Vertical" H 9350 9250 50  0001 C CNN
+F 3 "~" H 9350 9250 50  0001 C CNN
+	1    9350 9250
+	1    0    0    -1
+$EndComp
+Text GLabel 9550 9250 2    50   Input ~ 0
+RGB_DIN
+Wire Wire Line
+	9550 9150 9800 9150
+Wire Wire Line
+	9550 9350 9800 9350
+$Comp
+L power:+5V #PWR0141
+U 1 1 5EFB2986
+P 9800 9150
+F 0 "#PWR0141" H 9800 9000 50  0001 C CNN
+F 1 "+5V" V 9815 9278 50  0000 L CNN
+F 2 "" H 9800 9150 50  0001 C CNN
+F 3 "" H 9800 9150 50  0001 C CNN
+	1    9800 9150
+	0    1    1    0
+$EndComp
+$Comp
+L power:GND #PWR0142
+U 1 1 5EFB470E
+P 9800 9350
+F 0 "#PWR0142" H 9800 9100 50  0001 C CNN
+F 1 "GND" V 9805 9222 50  0000 R CNN
+F 2 "" H 9800 9350 50  0001 C CNN
+F 3 "" H 9800 9350 50  0001 C CNN
+	1    9800 9350
+	0    -1   -1   0
+$EndComp
+NoConn ~ 1400 14450
+NoConn ~ 15000 6600
 $EndSCHEMATC
