File: pcbV2/_autosave-keypadV2.sch (KiCad schematic (older format))
At the start: 73 parts, among them J1 Conn_01x02_Female, J2 USB_C_Receptacle, J3 Conn_01x03_Male, Q1 Q_NMOS_GSD, SW1 SW_Push, SW10 SW_Push, SW11 SW_Push, SW12 SW_Push, SW13 SW_SPDT, SW14 SW_Push, SW15 SW_Push, SW16 SW_Push, SW17 SW_DIP_x03, SW2 SW_Push, SW3 SW_Push, SW4 SW_Push, SW5 SW_Push, SW6 SW_Push, SW7 SW_Push, SW8 SW_Push, SW9 SW_Push, U1 Teensy4.0, U2 Waveshare_OLED_RGB

Commit message: basic layout v1
Connections:
- net RGB_DIN: now also Q1.3 (D), R3.2, R5.2
Changed lines of the file:
@@
 	6250 10000 7250 10000
 Wire Wire Line
-	7250 10000 7250 9450
+	7250 10000 7250 9700
 Text Notes 6000 10250 0    50   ~ 0
 *Option to put 220-470ohm (close to DIN)
@@
 	1    0    0    -1
 $EndComp
-Text GLabel 9550 9250 2    50   Input ~ 0
-RGB_DIN
 Wire Wire Line
 	9550 9150 9800 9150
@@
 NoConn ~ 1400 14450
 NoConn ~ 15000 6600
+Text GLabel 9550 9250 2    50   Input ~ 0
+RGB_DIN
+Wire Wire Line
+	7250 9700 7650 9700
+Connection ~ 7250 9700
+Wire Wire Line
+	7250 9700 7250 9450
+Text GLabel 7650 9700 2    50   Input ~ 0
+RGB_DIN
 $EndSCHEMATC
