File: pcbV2/_autosave-keypadV2.sch (KiCad schematic (older format))
At the start: 74 parts, among them J1 Conn_01x02_Female, J2 USB_C_Receptacle, J3 Conn_01x03_Male, Q1 Q_NMOS_GSD, SW1 SW_Push, SW10 SW_Push, SW11 SW_Push, SW12 SW_Push, SW13 SW_SPDT, SW14 SW_Push, SW15 SW_Push, SW16 SW_Push, SW17 SW_DIP_x03, SW2 SW_Push, SW3 SW_Push, SW4 SW_Push, SW5 SW_Push, SW6 SW_Push, SW7 SW_Push, SW8 SW_Push, SW9 SW_Push, U1 Teensy4.0, U2 Waveshare_OLED_RGB

Commit message: started layout of daughterboard
Parts:
- R6: footprint (none) -> Resistor_SMD:R_1206_3216Metric_Pad1.42x1.75mm_HandSolder
Changed lines of the file:
@@
 F 0 "R6" V 9043 10550 50  0000 C CNN
 F 1 "JUMPER" V 9134 10550 50  0000 C CNN
-F 2 "" V 9180 10550 50  0001 C CNN
+F 2 "Resistor_SMD:R_1206_3216Metric_Pad1.42x1.75mm_HandSolder" V 9180 10550 50  0001 C CNN
 F 3 "~" H 9250 10550 50  0001 C CNN
 	1    9250 10550
