File: pcbV2/keypadV2.sch (KiCad schematic (older format))
At the start: 72 parts

Commit message: start pcb layout
Parts:
- C1, C10, C11, C12, C13, C14, C15, C16, C2, C3, C4, C5, C6, C7, C8, C9: renamed from C?; footprint (none) -> Capacitor_SMD:C_1206_3216Metric_Pad1.42x1.75mm_HandSolder
- D1, D10, D11, D12, D2, D3, D4, D5, D6, D7, D8, D9: renamed from D?; footprint (none) -> Diode_SMD:D_SOD-323_HandSoldering
- D13: renamed from D?; footprint (none) -> LED_SMD:LED_1206_3216Metric_Pad1.42x1.75mm_HandSolder
- J1: renamed from J?; footprint (none) -> Connector_PinHeader_2.00mm:PinHeader_1x02_P2.00mm_Vertical
- Q1: renamed from Q?; footprint (none) -> Package_TO_SOT_SMD:SOT-23
- R1, R2, R3, R4, R5: renamed from R?; footprint (none) -> Resistor_SMD:R_1206_3216Metric_Pad1.42x1.75mm_HandSolder
- SW1, SW10, SW11, SW12, SW2, SW3, SW4, SW5, SW6, SW7, SW8, SW9: renamed from SW?; footprint (none) -> keyswitches:Kailh_socket_MX
- SW13: renamed from SW?; footprint (none) -> Connector_PinHeader_2.54mm:PinHeader_1x03_P2.54mm_Vertical
- U2: renamed from U?; footprint (none) -> Connector_PinHeader_2.54mm:PinHeader_1x07_P2.54mm_Vertical
- gave numbers to parts that had none: 22
Other:
- moved on the sheet: D13, R1, SW13, SW14
