File: pcbV2/keypadV2.sch (KiCad schematic (older format))
At the start: 59 parts, among them J1 Conn_01x02_Female, J2 USB_C_Receptacle, J3 Conn_01x03_Male, J6 Conn_01x03_Male, Q1 Q_NMOS_GSD, Q2 Q_NMOS_GSD, SW1 SW_Push, SW10 SW_Push, SW11 SW_Push, SW12 SW_Push, SW13 SW_SPDT, SW14 SW_Push, SW15 SW_Push, SW16 SW_Push, SW17 SW_DIP_x03, SW2 SW_Push, SW3 SW_Push, SW4 SW_Push, SW5 SW_Push, SW6 SW_Push, SW7 SW_Push, SW8 SW_Push, SW9 SW_Push, U1 Teensy4.0, U2 Waveshare_OLED_RGB

Commit message: started rewiring
Parts:
- removed J1: Conn_01x02_Female, Connector_PinHeader_2.00mm:PinHeader_1x02_P2.00mm_Vertical, symbol Connector:Conn_01x02_Female
- removed J2: USB_C_Receptacle, custom:USB_C_REDUCED_UJ31-CH-G2, symbol Connector:USB_C_Receptacle
- removed R4: R_SHIELD, Resistor_SMD:R_1206_3216Metric_Pad1.42x1.75mm_HandSolder, symbol Device:R
- removed SW13: SW_SPDT, Connector_PinHeader_2.54mm:PinHeader_1x03_P2.54mm_Vertical, symbol Switch:SW_SPDT
Connections:
- no-connect marks 47 -> 34
Other:
- note removed: "*Optional to connect shield to GND"
- note removed: "USB Data Breakouts"
- note removed: "USB-C Port"
Changed lines of the file:
@@
-$EndComp
-$Comp
-L Switch:SW_SPDT SW13
-U 1 1 5EF765BD
-P 13900 9000
-F 0 "SW13" H 13900 9285 50  0000 C CNN
-F 1 "SW_SPDT" H 13900 9194 50  0000 C CNN
-F 2 "Connector_PinHeader_2.54mm:PinHeader_1x03_P2.54mm_Vertical" H 13900 9000 50  0001 C CNN
-F 3 "~" H 13900 9000 50  0001 C CNN
-	1    13900 9000
-	1    0    0    -1
 $EndComp
 $Comp
@@
 	1    13900 11950
 	1    0    0    -1
-$EndComp
-$Comp
-L Connector:USB_C_Receptacle J2
-U 1 1 5EF7AA75
-P 18650 11500
-F 0 "J2" H 18220 11197 50  0000 R CNN
-F 1 "USB_C_Receptacle" H 18220 11288 50  0000 R CNN
-F 2 "custom:USB_C_REDUCED_UJ31-CH-G2" H 18800 11500 50  0001 C CNN
-F 3 "https://www.usb.org/sites/default/files/documents/usb_type-c.zip" H 18800 11500 50  0001 C CNN
-	1    18650 11500
-	-1   0    0    1
 $EndComp
 $Comp
@@
 	0    1    1    0
 $EndComp
-NoConn ~ 18050 10200
-NoConn ~ 18050 10300
-$Comp
-L Device:R R4
-U 1 1 5F08CE6B
-P 19400 9600
-F 0 "R4" V 19193 9600 50  0000 C CNN
-F 1 "R_SHIELD" V 19284 9600 50  0000 C CNN
-F 2 "Resistor_SMD:R_1206_3216Metric_Pad1.42x1.75mm_HandSolder" V 19330 9600 50  0001 C CNN
-F 3 "~" H 19400 9600 50  0001 C CNN
-	1    19400 9600
-	0    1    1    0
-$EndComp
-Wire Wire Line
-	19250 9600 18950 9600
-Wire Wire Line
-	18950 9600 18950 9900
-$Comp
-L power:GND #PWR0125
-U 1 1 5F092F41
-P 18650 9600
-F 0 "#PWR0125" H 18650 9350 50  0001 C CNN
-F 1 "GND" H 18655 9427 50  0000 C CNN
-F 2 "" H 18650 9600 50  0001 C CNN
-F 3 "" H 18650 9600 50  0001 C CNN
-	1    18650 9600
-	-1   0    0    1
-$EndComp
-Wire Wire Line
-	18650 9900 18650 9600
-NoConn ~ 18050 11400
-NoConn ~ 18050 11500
-NoConn ~ 18050 11100
-NoConn ~ 18050 11200
-NoConn ~ 18050 10800
-NoConn ~ 18050 10900
-NoConn ~ 18050 10500
-NoConn ~ 18050 10600
-NoConn ~ 18050 12200
-NoConn ~ 18050 12300
-$Comp
-L power:GND #PWR0126
-U 1 1 5F0BF5B3
-P 19750 9600
-F 0 "#PWR0126" H 19750 9350 50  0001 C CNN
-F 1 "GND" H 19755 9427 50  0000 C CNN
-F 2 "" H 19750 9600 50  0001 C CNN
-F 3 "" H 19750 9600 50  0001 C CNN
-	1    19750 9600
-	-1   0    0    1
-$EndComp
-Wire Wire Line
-	19750 9600 19550 9600
-Text GLabel 17800 11700 0    50   Input ~ 0
-USB_DATA+
-Text GLabel 17800 11800 0    50   Input ~ 0
-USB_DATA+
-Text GLabel 17800 11900 0    50   Input ~ 0
-USB_DATA-
-Text GLabel 17800 12000 0    50   Input ~ 0
-USB_DATA-
-Text GLabel 17800 12500 0    50   Input ~ 0
-USB_VBUS
-Wire Wire Line
-	18050 11700 17800 11700
-Wire Wire Line
-	18050 11800 17800 11800
-Wire Wire Line
-	18050 11900 17800 11900
-Wire Wire Line
-	18050 12000 17800 12000
-Wire Wire Line
-	18050 12500 17800 12500
-Text Notes 19250 9850 0    50   ~ 0
-*Optional to connect shield to GND
-Wire Wire Line
-	14100 8900 14400 8900
-$Comp
-L power:+5V #PWR0127
-U 1 1 5F0D8397
-P 14400 8900
-F 0 "#PWR0127" H 14400 8750 50  0001 C CNN
-F 1 "+5V" V 14415 9028 50  0000 L CNN
-F 2 "" H 14400 8900 50  0001 C CNN
-F 3 "" H 14400 8900 50  0001 C CNN
-	1    14400 8900
-	0    1    1    0
-$EndComp
-Wire Wire Line
-	13700 9000 13550 9000
-Text GLabel 13550 9000 0    50   Input ~ 0
-USB_VBUS
 Text GLabel 8750 4850 0    50   Input ~ 0
 ON_OFF
@@
 	3600 9250 3400 9250
 Connection ~ 3400 9250
-$Comp
-L Connector:Conn_01x02_Female J1
-U 1 1 5F17D824
-P 18550 7900
-F 0 "J1" H 18578 7876 50  0000 L CNN
-F 1 "Conn_01x02_Female" H 18578 7785 50  0000 L CNN
-F 2 "Connector_PinHeader_2.00mm:PinHeader_1x02_P2.00mm_Vertical" H 18550 7900 50  0001 C CNN
-F 3 "~" H 18550 7900 50  0001 C CNN
-	1    18550 7900
-	1    0    0    -1
-$EndComp
-Text GLabel 18200 7900 0    50   Input ~ 0
-USB_DATA+
-Text GLabel 18200 8000 0    50   Input ~ 0
-USB_DATA-
-Wire Wire Line
-	18350 7900 18200 7900
-Wire Wire Line
-	18350 8000 18200 8000
 Wire Wire Line
 	5650 11350 6050 11350
@@
 Text Notes 13300 8400 0    118  ~ 0
 Power Controls
-Text Notes 17650 7650 0    118  ~ 0
-USB Data Breakouts
 Text Notes 3650 3500 0    118  ~ 0
 Display
 Text Notes 4850 7600 0    118  ~ 0
 Addressable RGBs
-Text Notes 18050 9100 0    118  ~ 0
-USB-C Port
 Text Notes 2500 8350 0    79   ~ 0
 RGB Data Logic Level Shifter \n(Individual Backlighting)
@@
 $EndComp
 NoConn ~ 5050 11350
-NoConn ~ 14100 9100
 Text GLabel 3000 11050 2    50   Input ~ 0
 RGB_DIN

Commit message: update
Parts:
- C13, C14, C15, C16: value 1000uF -> 1uF
Changed lines of the file:
@@
 P 5050 11800
 F 0 "C13" H 5165 11846 50  0000 L CNN
-F 1 "1000uF" H 5165 11755 50  0000 L CNN
+F 1 "1uF" H 5165 11755 50  0000 L CNN
 F 2 "Capacitor_SMD:C_1206_3216Metric_Pad1.42x1.75mm_HandSolder" H 5088 11650 50  0001 C CNN
 F 3 "~" H 5050 11800 50  0001 C CNN
@@
 P 6050 11800
 F 0 "C14" H 6165 11846 50  0000 L CNN
-F 1 "1000uF" H 6165 11755 50  0000 L CNN
+F 1 "1uF" H 6165 11755 50  0000 L CNN
 F 2 "Capacitor_SMD:C_1206_3216Metric_Pad1.42x1.75mm_HandSolder" H 6088 11650 50  0001 C CNN
 F 3 "~" H 6050 11800 50  0001 C CNN
@@
 P 7050 11800
 F 0 "C15" H 7165 11846 50  0000 L CNN
-F 1 "1000uF" H 7165 11755 50  0000 L CNN
+F 1 "1uF" H 7165 11755 50  0000 L CNN
 F 2 "Capacitor_SMD:C_1206_3216Metric_Pad1.42x1.75mm_HandSolder" H 7088 11650 50  0001 C CNN
 F 3 "~" H 7050 11800 50  0001 C CNN
@@
 P 8050 11800
 F 0 "C16" H 8165 11846 50  0000 L CNN
-F 1 "1000uF" H 8165 11755 50  0000 L CNN
+F 1 "1uF" H 8165 11755 50  0000 L CNN
 F 2 "Capacitor_SMD:C_1206_3216Metric_Pad1.42x1.75mm_HandSolder" H 8088 11650 50  0001 C CNN
 F 3 "~" H 8050 11800 50  0001 C CNN
